Commit message: fix_filepath and directory

File: src/gazebo_simulation/urdf/armmyRobot2.urdf (robot description, URDF)
Before this commit: robot urdf_tutorial, 3 links, 2 joints
Links:
- link W_L: geometry collision mesh filename=package://gazebo_simulation/meshes/W_L.STL; visual mesh filename=package://gazebo_simulation/meshes/W_L.STL
- link W_R: geometry collision mesh filename=package://gazebo_simulation/meshes/W_R.STL; visual mesh filename=package://gazebo_simulation/meshes/W_R.STL
- link base_link: geometry collision mesh filename=package://gazebo_simulation/meshes/base_link.STL; visual mesh filename=package://gazebo_simulation/meshes/base_link.STL

Commit message: still stuck at spawn robot to gazebo

File: src/gazebo_simulation/urdf/armmyRobot2.urdf (robot description, URDF)
Before this commit: robot urdf_tutorial, 3 links, 2 joints
Joints:
- joint W_L_joint: origin xyz=0.006 -0.02 0.008 rpy=-3.1416 0.85417 1.5708 -> xyz=0.006 -0.02 0.008 rpy=0 0 -1.571
- joint W_R_joint: origin xyz=-0.086 -0.02 0.008 rpy=0 0.38986 1.5708 -> xyz=-0.086 -0.02 0.008 rpy=0 0 1.571

File: src/gazebo_simulation/urdf/rs_robot.urdf (robot description, URDF)
Before this commit: robot rs_robot, 10 links, 9 joints
Links:
- link base_link: geometry collision mesh filename=package://gazebo_simulation/models/rs_robot/meshes/STL/base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; visual mesh filename=package://gazebo_simulation/models/rs_robot/meshes/DAE/base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
- link fl_steering_link: geometry collision mesh filename=package://gazebo_simulation/models/rs_robot/meshes/STL/susp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; visual mesh filename=package://gazebo_simulation/models/rs_robot/meshes/DAE/susp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
- link fl_wheel_link: geometry collision mesh filename=package://gazebo_simulation/models/rs_robot/meshes/STL/whee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; visual mesh filename=package://gazebo_simulation/models/rs_robot/meshes/DAE/whee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
- link fr_steering_link: geometry collision mesh filename=package://gazebo_simulation/models/rs_robot/meshes/STL/susp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; visual mesh filename=package://gazebo_simulation/models/rs_robot/meshes/DAE/susp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
- link fr_wheel_link: geometry collision mesh filename=package://gazebo_simulation/models/rs_robot/meshes/STL/whee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; visual mesh filename=package://gazebo_simulation/models/rs_robot/meshes/DAE/whee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
- link rl_steering_link: geometry collision mesh filename=package://gazebo_simulation/models/rs_robot/meshes/STL/susp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; visual mesh filename=package://gazebo_simulation/models/rs_robot/meshes/DAE/susp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
- link rl_wheel_link: geometry collision mesh filename=package://gazebo_simulation/models/rs_robot/meshes/STL/whee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; visual mesh filename=package://gazebo_simulation/models/rs_robot/meshes/DAE/whee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
- link rr_steering_link: geometry collision mesh filename=package://gazebo_simulation/models/rs_robot/meshes/STL/susp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; visual mesh filename=package://gazebo_simulation/models/rs_robot/meshes/DAE/susp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
- link rr_wheel_link: geometry collision mesh filename=package://gazebo_simulation/models/rs_robot/meshes/STL/whee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; visual mesh filename=package://gazebo_simulation/models/rs_robot/meshes/DAE/whee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
