Commit message: before sleep, next obj: create track map

File: src/gazebo_simulation/urdf/armmyRobot3_cam_gazebo.urdf (robot description, URDF)
Before this commit: robot ArmmyRobotURDF3, 6 links, 5 joints
Joints:
- joint camera_joint: origin xyz=-0.04 -0.085 0.08 rpy=0 0 -1.571 -> xyz=-0.04 -0.085 0.12 rpy=0 0.2 -1.571

Commit message: adjust camera position

File: src/gazebo_simulation/urdf/armmyRobot3_cam_gazebo.urdf (robot description, URDF)
Before this commit: robot ArmmyRobotURDF3, 6 links, 5 joints
Joints:
- joint camera_joint: origin xyz=-0.04 -0.085 0.12 rpy=0 0.2 -1.571 -> xyz=-0.04 -0.085 0.12 rpy=0 0.4 -1.571
